Commit message: Added move_base to scout for basic navigation. A laser is being used for scanning the environment for now - TODO For ground truth we're using world position provided by gazebo - TODO Removed front wheels and replaced with castor wheel - TODO after integrating ros_control

File: src/ssam_simulation/models/scout/parameter.xacro (robot description, xacro)
@@ -13,3 +13,7 @@
   <xacro:property name="torque_wheel" value="10" />
   <xacro:property name="L_wheel" value="0.1788" />
+  <!-- Parameters for the Hukoyu Laser -->
+  <xacro:property name="x_hokuyo" value="0.1" />
+  <xacro:property name="y_hokuyo" value="0.1" />
+  <xacro:property name="z_hokuyo" value="0.1" />
 </robot>

File: src/ssam_simulation/models/scout/scout.xacro (robot description, xacro)
@@ -35,4 +35,26 @@
       <geometry>
         <box size="${x_chassis} ${y_chassis} ${z_chassis}"/>
+      </geometry>
+    </visual>
+    <collision name='caster_collision'>
+      <origin xyz="${-(r_wheel/2)+x_chassis/2} 0 ${-z_chassis/2}" rpy=" 0 0 0"/>
+      <geometry>
+        <sphere radius="${r_wheel/2}"/>
+      </geometry>
+      <surface>
+        <friction>
+          <ode>
+            <mu>0</mu>
+            <mu2>0</mu2>
+            <slip1>1.0</slip1>
+            <slip2>1.0</slip2>
+          </ode>
+        </friction>
+      </surface>
+    </collision>
+    <visual name='caster_visual'>
+      <origin xyz="${-(r_wheel/2)+x_chassis/2} 0 ${-z_chassis/2}" rpy=" 0 0 0"/>
+      <geometry>
+        <sphere radius="${r_wheel/2}"/>
       </geometry>
     </visual>
@@ -99,64 +121,4 @@
     </inertial>
   </link>
-  <link name="left_front_wheel">
-    <collision name="collision">
-      <origin xyz="0 0 0" rpy="0 1.5707 1.5707"/>
-      <geometry>
-        <cylinder radius="${r_wheel}" length="${h_wheel}"/>
-      </geometry>
-      <surface>
-        <friction>
-          <ode>
-            <mu>1.0</mu>
-            <mu2>1.0</mu2>
-            <slip1>0.0</slip1>
-            <slip2>0.0</slip2>
-          </ode>
-        </friction>
-      </surface>
-    </collision>
-    <visual name="left_wheel_visual">
-      <origin xyz="0 0 0" rpy="0 1.5707 1.5707"/>
-      <geometry>
-        <cylinder radius="${r_wheel}" length="${h_wheel}"/>
-      </geometry>
-    </visual>
-    <inertial>
-      <origin xyz="0 0 0" rpy="0 1.5707 1.5707"/>
-      <mass value="${m_wheel}"/>
-      <cylinder_inertia m="${m_wheel}" r="${r_wheel}" h="${h_wheel}"/>
-      <xacro:cylinder_inertia m="${m_wheel}" r="${r_wheel}" h="${h_wheel}"/>
-    </inertial>
-  </link>
-  <link name="right_front_wheel">
-    <collision name="collision">
-      <origin xyz="0 0 0" rpy="0 1.5707 1.5707"/>
-      <geometry>
-        <cylinder radius="${r_wheel}" length="${h_wheel}"/>
-      </geometry>
-      <surface>
-        <friction>
-          <ode>
-            <mu>1.0</mu>
-            <mu2>1.0</mu2>
-            <slip1>0.0</slip1>
-            <slip2>0.0</slip2>
-          </ode>
-        </friction>
-      </surface>
-    </collision>
-    <visual name="right_wheel_visual">
-      <origin xyz="0 0 0" rpy="0 1.5707 1.5707"/>
-      <geometry>
-        <cylinder radius="${r_wheel}" length="${h_wheel}"/>
-      </geometry>
-    </visual>
-    <inertial>
-      <origin xyz="0 0 0" rpy="0 1.5707 1.5707"/>
-      <mass value="${m_wheel}"/>
-      <cylinder_inertia m="${m_wheel}" r="${r_wheel}" h="${h_wheel}"/>
-      <xacro:cylinder_inertia m="${m_wheel}" r="${r_wheel}" h="${h_wheel}"/>
-    </inertial>
-  </link>
   <!-- Set joints for the wheels which can be controlled over ROS -->
   <joint type="continuous" name="left_back_wheel_hinge">
@@ -176,19 +138,30 @@
     <joint_properties damping="0.0" friction="0.0"/>
   </joint>
-   <joint type="continuous" name="left_front_wheel_hinge">
-    <origin xyz="${x_chassis/3} ${y_chassis/2+h_wheel/2} ${r_wheel/2-z_chassis/2}" rpy="0 0 0"/>
-    <child link="left_front_wheel"/>
+  <!-- Add a Hokuyo Laser -->
+  <link name="laser_link">
+    <collision>
+      <origin xyz="0 0 0" rpy="0 0 0"/>
+      <geometry>
+		<box size="${x_hokuyo} ${y_hokuyo} ${z_hokuyo}"/>
+      </geometry>
+    </collision>
+    <visual>
+      <origin xyz="0 0 0" rpy="0 0 0"/>
+      <geometry>
+        <!-- <mesh filename="package://rrbot_description/meshes/hokuyo.dae"/> -->
+        <box size="${x_hokuyo} ${y_hokuyo} ${z_hokuyo}"/>
+      </geometry>
+    </visual>
+    <inertial>
+      <mass value="1e-5" />
+      <origin xyz="0 0 0" rpy="0 0 0"/>
+      <inertia ixx="1e-6" ixy="0" ixz="0" iyy="1e-6" iyz="0" izz="1e-6" />
+    </inertial>
+  </link>
+  <joint name="hokuyo_joint" type="fixed">
+    <axis xyz="0 1 0" />
+    <origin xyz="0 0 ${z_chassis/2 + z_hokuyo/2}" rpy="0 0 0"/>
     <parent link="base_link"/>
-    <axis xyz="0 1 0" rpy="0 0 0"/>
-    <limit effort="100" velocity="100"/>
-    <joint_properties damping="0.0" friction="0.0"/>
-  </joint>
-  <joint type="continuous" name="right_front_wheel_hinge">
-    <origin xyz="${x_chassis/3} ${-y_chassis/2-h_wheel/2} ${r_wheel/2-z_chassis/2}" rpy="0 0 0"/>
-    <child link="right_front_wheel"/>
-    <parent link="base_link"/>
-    <axis xyz="0 1 0" rpy="0 0 0"/>
-    <limit effort="100" velocity="100"/>
-    <joint_properties damping="0.0" friction="0.0"/>
+    <child link="laser_link"/>
   </joint>
  </robot>

Commit message: Use stereo camera for navigation instead of laser.

File: src/ssam_simulation/models/scout/parameter.xacro (robot description, xacro)
@@ -13,7 +13,13 @@
   <xacro:property name="torque_wheel" value="10" />
   <xacro:property name="L_wheel" value="0.1788" />
-  <!-- Parameters for the Hukoyu Laser -->
-  <xacro:property name="x_hokuyo" value="0.1" />
-  <xacro:property name="y_hokuyo" value="0.1" />
-  <xacro:property name="z_hokuyo" value="0.1" />
+  <!-- Parameters for the stereo camera-->
+  <xacro:property name="x_camera" value="0.2" />
+  <xacro:property name="y_camera" value="0" />
+  <xacro:property name="z_camera" value="${z_chassis/2 + h_camera/2}"/>
+  <xacro:property name="w_camera" value="0.1" />
+  <xacro:property name="l_camera" value="0.1" />
+  <xacro:property name="h_camera" value="0.1" />
+  <xacro:property name="camera_res_w" value="1280" />
+  <xacro:property name="camera_res_h" value="800" />
+  <xacro:property name="camera_fov" value="1.22173" />
 </robot>

File: src/ssam_simulation/models/scout/scout.xacro (robot description, xacro)
@@ -89,10 +89,9 @@
   <xacro:scout_wheel prefix="right_back" xReflect="-1" yReflect="-1"/>
   <xacro:scout_wheel prefix="right_front" xReflect="1" yReflect="-1"/>
-  <!-- Add a Hokuyo Laser -->
-  <link name="laser_link">
+  <link name="camera_link">
     <collision>
       <origin xyz="0 0 0" rpy="0 0 0"/>
       <geometry>
-		<box size="${x_hokuyo} ${y_hokuyo} ${z_hokuyo}"/>
+		<box size="${l_camera} ${w_camera} ${h_camera}"/>
       </geometry>
     </collision>
@@ -100,6 +99,5 @@
       <origin xyz="0 0 0" rpy="0 0 0"/>
       <geometry>
-        <!-- <mesh filename="package://rrbot_description/meshes/hokuyo.dae"/> -->
-        <box size="${x_hokuyo} ${y_hokuyo} ${z_hokuyo}"/>
+        <box size="${l_camera} ${w_camera} ${h_camera}"/>
       </geometry>
     </visual>
@@ -110,9 +108,15 @@
     </inertial>
   </link>
-  <joint name="hokuyo_joint" type="fixed">
-    <axis xyz="0 1 0" />
-    <origin xyz="0 0 ${z_chassis/2 + z_hokuyo/2}" rpy="0 0 0"/>
+  <joint name="camera_joint" type="fixed">
+    <origin xyz="${x_camera} ${y_camera} ${z_camera}" rpy="0 0 0"/>
     <parent link="base_link"/>
-    <child link="laser_link"/>
+    <child link="camera_link"/>
+  </joint>
+  <link name="camera_link_optical">
+  </link>
+  <joint name="camera_optical_joint" type="fixed">
+    <origin xyz="0 0 0" rpy="${-pi/2} 0 ${-pi/2}"/>
+    <parent link="camera_link"/>
+    <child link="camera_link_optical"/>
   </joint>
   <transmission name="left_back_wheel_transmission">

Commit message: Reduce camera fps from 60 to 5

File: src/ssam_simulation/models/scout/parameter.xacro (robot description, xacro)
@@ -23,3 +23,4 @@
   <xacro:property name="camera_res_h" value="800" />
   <xacro:property name="camera_fov" value="1.22173" />
+  <xacro:property name="camera_fps" value="5.0" />
 </robot>
